File: CPU.sch (KiCad schematic (older format))
At the start: 25 parts, among them J1 10.0402_LCD_RGB_CON_WJQ, SW1 11.0101_SW-A03-08, U1 08.0001_F1C200S, Y1 07.0403_Crystal_24M_3225

Commit message: 优化封装外形丝印，PCB进行拼板处理
Parts:
- C1, C12, C2, C5: value 03.0016_C0603_10uF -> 03.4004_C0603_10uF; footprint Capacitor_SMD:C_0603_1608Metric -> 0WJQ:C_0603_WJQ; symbol 0WJQ:03.0016_C0603_10uF -> 0WJQ:03.4004_C0603_10uF; 编码 03.0016 -> 03.4004
- C10, C13, C14, C15, C16, C17, C18, C3, C4, C6, C7, C8, C9: footprint Capacitor_SMD:C_0402_1005Metric -> 0WJQ:C_0402_WJQ
- C11: value 03.0011_C0603_1uF -> 03.4004_C0603_10uF; footprint Capacitor_SMD:C_0603_1608Metric -> 0WJQ:C_0603_WJQ; symbol 0WJQ:03.0011_C0603_1uF -> 0WJQ:03.4004_C0603_10uF; 参数 1uF -> 10uF; 编码 03.0011 -> 03.4004; 规格 1uF,16V,K,0603,,X7R -> 10uF,16V,K,0603,X5R
- R1, R2, R3: footprint Resistor_SMD:R_0402_1005Metric -> 0WJQ:R_0402_WJQ
Changed lines of the file:
@@
 $EndComp
 $Comp
-L 0WJQ:03.0016_C0603_10uF C?
+L 0WJQ:03.4004_C0603_10uF C?
 U 1 1 5E438D56
 P 4300 6450
 AR Path="/5E3A4AC6/5E438D56" Ref="C?"  Part="1"
 AR Path="/5E3A4A8E/5E438D56" Ref="C12"  Part="1"
+AR Path="/5E438D56" Ref="C12"  Part="1"
 F 0 "C12" H 4392 6496 50  0000 L CNN
-F 1 "03.0016_C0603_10uF" H 4310 6370 50  0001 L CNN
-F 2 "Capacitor_SMD:C_0603_1608Metric" H 3700 6400 50  0001 C CNN
+F 1 "03.4004_C0603_10uF" H 4310 6370 50  0001 L CNN
+F 2 "0WJQ:C_0603_WJQ" H 3700 6400 50  0001 C CNN
 F 3 "~" H 4300 6450 50  0001 C CNN
 F 4 "贴片瓷片电容" H 4300 6450 50  0001 C CNN "分类"
-F 5 "03.0016" H 4300 6450 50  0001 C CNN "编码"
+F 5 "03.4004" H 4300 6450 50  0001 C CNN "编码"
 F 6 "10uF,16V,K,0603,X5R" H 4300 6450 50  0001 C CNN "规格"
 F 7 "10uF" H 4392 6405 50  0000 L CNN "参数"
@@
 F 0 "C13" H 4742 6496 50  0000 L CNN
 F 1 "03.0009_C0402_100nF" H 4660 6270 50  0001 L CNN
-F 2 "Capacitor_SMD:C_0402_1005Metric" H 4700 6400 50  0001 C CNN
+F 2 "0WJQ:C_0402_WJQ" H 4700 6400 50  0001 C CNN
 F 3 "~" H 4650 6450 50  0001 C CNN
 F 4 "贴片瓷片电容" H 4650 6450 50  0001 C CNN "分类"
@@
 F 0 "R1" H 4700 6743 50  0000 C CNN
 F 1 "02.0026_R0402_2K_1%" H 4550 7140 50  0001 L BNN
-F 2 "Resistor_SMD:R_0402_1005Metric" H 4500 6710 50  0001 L BNN
+F 2 "0WJQ:R_0402_WJQ" H 4500 6710 50  0001 L BNN
 F 3 "" H 4500 6810 50  0001 L BNN
 F 4 "贴片电阻" H 4700 6950 50  0001 C CNN "分类"
@@
 F 0 "R2" H 5300 6743 50  0000 C CNN
 F 1 "02.0026_R0402_2K_1%" H 5150 7140 50  0001 L BNN
-F 2 "Resistor_SMD:R_0402_1005Metric" H 5100 6710 50  0001 L BNN
+F 2 "0WJQ:R_0402_WJQ" H 5100 6710 50  0001 L BNN
 F 3 "" H 5100 6810 50  0001 L BNN
 F 4 "贴片电阻" H 5300 6950 50  0001 C CNN "分类"
@@
 F 0 "C14" H 4842 7196 50  0000 L CNN
 F 1 "03.0009_C0402_100nF" H 4760 6970 50  0001 L CNN
-F 2 "Capacitor_SMD:C_0402_1005Metric" H 4800 7100 50  0001 C CNN
+F 2 "0WJQ:C_0402_WJQ" H 4800 7100 50  0001 C CNN
 F 3 "~" H 4750 7150 50  0001 C CNN
 F 4 "贴片瓷片电容" H 4750 7150 50  0001 C CNN "分类"
@@
 F 0 "C15" H 5392 7196 50  0000 L CNN
 F 1 "03.0009_C0402_100nF" H 5310 6970 50  0001 L CNN
-F 2 "Capacitor_SMD:C_0402_1005Metric" H 5350 7100 50  0001 C CNN
+F 2 "0WJQ:C_0402_WJQ" H 5350 7100 50  0001 C CNN
 F 3 "~" H 5300 7150 50  0001 C CNN
 F 4 "贴片瓷片电容" H 5300 7150 50  0001 C CNN "分类"
@@
 Connection ~ 4300 6700
 $Comp
-L 0WJQ:03.0016_C0603_10uF C?
+L 0WJQ:03.4004_C0603_10uF C?
 U 1 1 5E449C11
 P 1250 5550
 AR Path="/5E3A4AC6/5E449C11" Ref="C?"  Part="1"
 AR Path="/5E3A4A8E/5E449C11" Ref="C1"  Part="1"
+AR Path="/5E449C11" Ref="C1"  Part="1"
 F 0 "C1" H 1342 5596 50  0000 L CNN
-F 1 "03.0016_C0603_10uF" H 1260 5470 50  0001 L CNN
-F 2 "Capacitor_SMD:C_0603_1608Metric" H 650 5500 50  0001 C CNN
+F 1 "03.4004_C0603_10uF" H 1260 5470 50  0001 L CNN
+F 2 "0WJQ:C_0603_WJQ" H 650 5500 50  0001 C CNN
 F 3 "~" H 1250 5550 50  0001 C CNN
 F 4 "贴片瓷片电容" H 1250 5550 50  0001 C CNN "分类"
-F 5 "03.0016" H 1250 5550 50  0001 C CNN "编码"
+F 5 "03.4004" H 1250 5550 50  0001 C CNN "编码"
 F 6 "10uF,16V,K,0603,X5R" H 1250 5550 50  0001 C CNN "规格"
 F 7 "10uF" H 1342 5505 50  0000 L CNN "参数"
@@
 F 0 "C3" H 1692 5596 50  0000 L CNN
 F 1 "03.0009_C0402_100nF" H 1610 5370 50  0001 L CNN
-F 2 "Capacitor_SMD:C_0402_1005Metric" H 1650 5500 50  0001 C CNN
+F 2 "0WJQ:C_0402_WJQ" H 1650 5500 50  0001 C CNN
 F 3 "~" H 1600 5550 50  0001 C CNN
 F 4 "贴片瓷片电容" H 1600 5550 50  0001 C CNN "分类"
@@
 $EndComp
 $Comp
-L 0WJQ:03.0016_C0603_10uF C?
+L 0WJQ:03.4004_C0603_10uF C?
 U 1 1 5E44DE25
 P 1750 3000
 AR Path="/5E3A4AC6/5E44DE25" Ref="C?"  Part="1"
 AR Path="/5E3A4A8E/5E44DE25" Ref="C5"  Part="1"
+AR Path="/5E44DE25" Ref="C5"  Part="1"
 F 0 "C5" H 1842 3046 50  0000 L CNN
-F 1 "03.0016_C0603_10uF" H 1760 2920 50  0001 L CNN
-F 2 "Capacitor_SMD:C_0603_1608Metric" H 1150 2950 50  0001 C CNN
+F 1 "03.4004_C0603_10uF" H 1760 2920 50  0001 L CNN
+F 2 "0WJQ:C_0603_WJQ" H 1150 2950 50  0001 C CNN
 F 3 "~" H 1750 3000 50  0001 C CNN
 F 4 "贴片瓷片电容" H 1750 3000 50  0001 C CNN "分类"
-F 5 "03.0016" H 1750 3000 50  0001 C CNN "编码"
+F 5 "03.4004" H 1750 3000 50  0001 C CNN "编码"
 F 6 "10uF,16V,K,0603,X5R" H 1750 3000 50  0001 C CNN "规格"
 F 7 "10uF" H 1842 2955 50  0000 L CNN "参数"
@@
 F 0 "C8" H 2192 3046 50  0000 L CNN
 F 1 "03.0009_C0402_100nF" H 2110 2820 50  0001 L CNN
-F 2 "Capacitor_SMD:C_0402_1005Metric" H 2150 2950 50  0001 C CNN
+F 2 "0WJQ:C_0402_WJQ" H 2150 2950 50  0001 C CNN
 F 3 "~" H 2100 3000 50  0001 C CNN
 F 4 "贴片瓷片电容" H 2100 3000 50  0001 C CNN "分类"
@@
 	6050 1650 6300 1650
 $Comp
-L 0WJQ:03.0011_C0603_1uF C11
+L 0WJQ:03.4004_C0603_10uF C11
 U 1 1 5E4621A7
 P 3850 6450
+AR Path="/5E4621A7" Ref="C11"  Part="1"
+AR Path="/5E3A4A8E/5E4621A7" Ref="C11"  Part="1"
 F 0 "C11" H 3942 6496 50  0000 L CNN
-F 1 "03.0011_C0603_1uF" H 3860 6270 50  0001 L CNN
-F 2 "Capacitor_SMD:C_0603_1608Metric" H 3250 6400 50  0001 C CNN
+F 1 "03.4004_C0603_10uF" H 3860 6270 50  0001 L CNN
+F 2 "0WJQ:C_0603_WJQ" H 3250 6400 50  0001 C CNN
 F 3 "~" H 3850 6450 50  0001 C CNN
 F 4 "贴片瓷片电容" H 3850 6350 50  0001 C CNN "分类"
-F 5 "03.0011" H 3850 6350 50  0001 C CNN "编码"
-F 6 "1uF,16V,K,0603,,X7R" H 3850 6350 50  0001 C CNN "规格"
-F 7 "1uF" H 3942 6405 50  0000 L CNN "参数"
+F 5 "03.4004" H 3850 6350 50  0001 C CNN "编码"
+F 6 "10uF,16V,K,0603,X5R" H 3850 6350 50  0001 C CNN "规格"
+F 7 "10uF" H 3942 6405 50  0000 L CNN "参数"
 	1    3850 6450
 	1    0    0    -1
@@
 F 0 "R3" V 7404 1120 50  0000 L CNN
 F 1 "02.0008_R0402_10K_1%" H 7300 1240 50  0001 L BNN
-F 2 "Resistor_SMD:R_0402_1005Metric" H 7250 810 50  0001 L BNN
+F 2 "0WJQ:R_0402_WJQ" H 7250 810 50  0001 L BNN
 F 3 "" H 7250 910 50  0001 L BNN
 F 4 "贴片电阻" H 7450 1050 50  0001 C CNN "分类"
@@
 F 0 "C16" H 7542 1596 50  0000 L CNN
 F 1 "03.0001_C0402_1uF" H 7510 1220 50  0001 L CNN
-F 2 "Capacitor_SMD:C_0402_1005Metric" H 7450 1150 50  0001 C CNN
+F 2 "0WJQ:C_0402_WJQ" H 7450 1150 50  0001 C CNN
 F 3 "~" H 7450 1550 50  0001 C CNN
 F 4 "贴片瓷片电容" H 7550 1050 50  0001 C CNN "分类"
@@
 	7050 2150 7350 2150
 $Comp
-L 0WJQ:03.0016_C0603_10uF C?
+L 0WJQ:03.4004_C0603_10uF C?
 U 1 1 5E53E3CE
 P 1250 6850
 AR Path="/5E3A4AC6/5E53E3CE" Ref="C?"  Part="1"
 AR Path="/5E3A4A8E/5E53E3CE" Ref="C2"  Part="1"
+AR Path="/5E53E3CE" Ref="C2"  Part="1"
 F 0 "C2" H 1342 6896 50  0000 L CNN
-F 1 "03.0016_C0603_10uF" H 1260 6770 50  0001 L CNN
-F 2 "Capacitor_SMD:C_0603_1608Metric" H 650 6800 50  0001 C CNN
+F 1 "03.4004_C0603_10uF" H 1260 6770 50  0001 L CNN
+F 2 "0WJQ:C_0603_WJQ" H 650 6800 50  0001 C CNN
 F 3 "~" H 1250 6850 50  0001 C CNN
 F 4 "贴片瓷片电容" H 1250 6850 50  0001 C CNN "分类"
-F 5 "03.0016" H 1250 6850 50  0001 C CNN "编码"
+F 5 "03.4004" H 1250 6850 50  0001 C CNN "编码"
 F 6 "10uF,16V,K,0603,X5R" H 1250 6850 50  0001 C CNN "规格"
 F 7 "10uF" H 1342 6805 50  0000 L CNN "参数"
@@
 F 0 "C4" H 1692 6896 50  0000 L CNN
 F 1 "03.0009_C0402_100nF" H 1610 6670 50  0001 L CNN
-F 2 "Capacitor_SMD:C_0402_1005Metric" H 1650 6800 50  0001 C CNN
+F 2 "0WJQ:C_0402_WJQ" H 1650 6800 50  0001 C CNN
 F 3 "~" H 1600 6850 50  0001 C CNN
 F 4 "贴片瓷片电容" H 1600 6850 50  0001 C CNN "分类"
@@
 F 0 "C18" H 8492 5746 50  0000 L CNN
 F 1 "03.0003_C0402_10pF" H 8360 5470 50  0001 L CNN
-F 2 "Capacitor_SMD:C_0402_1005Metric" H 7800 5650 50  0001 C CNN
+F 2 "0WJQ:C_0402_WJQ" H 7800 5650 50  0001 C CNN
 F 3 "~" H 8400 5700 50  0001 C CNN
 F 4 "贴片瓷片电容" H 8350 5550 50  0001 C CNN "分类"
@@
 F 0 "C17" H 8092 5746 50  0000 L CNN
 F 1 "03.0003_C0402_10pF" H 7960 5470 50  0001 L CNN
-F 2 "Capacitor_SMD:C_0402_1005Metric" H 7400 5650 50  0001 C CNN
+F 2 "0WJQ:C_0402_WJQ" H 7400 5650 50  0001 C CNN
 F 3 "~" H 8000 5700 50  0001 C CNN
 F 4 "贴片瓷片电容" H 7950 5550 50  0001 C CNN "分类"
@@
 F 0 "C7" H 2092 6896 50  0000 L CNN
 F 1 "03.0009_C0402_100nF" H 2010 6670 50  0001 L CNN
-F 2 "Capacitor_SMD:C_0402_1005Metric" H 2050 6800 50  0001 C CNN
+F 2 "0WJQ:C_0402_WJQ" H 2050 6800 50  0001 C CNN
 F 3 "~" H 2000 6850 50  0001 C CNN
 F 4 "贴片瓷片电容" H 2000 6850 50  0001 C CNN "分类"
@@
 F 0 "C10" H 2492 6896 50  0000 L CNN
 F 1 "03.0009_C0402_100nF" H 2410 6670 50  0001 L CNN
-F 2 "Capacitor_SMD:C_0402_1005Metric" H 2450 6800 50  0001 C CNN
+F 2 "0WJQ:C_0402_WJQ" H 2450 6800 50  0001 C CNN
 F 3 "~" H 2400 6850 50  0001 C CNN
 F 4 "贴片瓷片电容" H 2400 6850 50  0001 C CNN "分类"
@@
 F 0 "C6" H 2092 5596 50  0000 L CNN
 F 1 "03.0009_C0402_100nF" H 2010 5370 50  0001 L CNN
-F 2 "Capacitor_SMD:C_0402_1005Metric" H 2050 5500 50  0001 C CNN
+F 2 "0WJQ:C_0402_WJQ" H 2050 5500 50  0001 C CNN
 F 3 "~" H 2000 5550 50  0001 C CNN
 F 4 "贴片瓷片电容" H 2000 5550 50  0001 C CNN "分类"
@@
 F 0 "C9" H 2492 5596 50  0000 L CNN
 F 1 "03.0009_C0402_100nF" H 2410 5370 50  0001 L CNN
-F 2 "Capacitor_SMD:C_0402_1005Metric" H 2450 5500 50  0001 C CNN
+F 2 "0WJQ:C_0402_WJQ" H 2450 5500 50  0001 C CNN
 F 3 "~" H 2400 5550 50  0001 C CNN
 F 4 "贴片瓷片电容" H 2400 5550 50  0001 C CNN "分类"
