File: Misc.sch (KiCad schematic (older format))
At the start: 23 parts, among them J2 10.0002_USB_Micro, J3 10.0001_Micro_SD_Card, J4 10.0201_PH2X15_2D54_V, J5 10.0002_USB_Micro, U4 09.0001_CP2104, U5 09.0303_GD5F1GQ4, U6 09.0302_W25Q128JVS

Commit message: 优化封装外形丝印，PCB进行拼板处理
Parts:
- C31: value 03.0011_C0603_1uF -> 03.4001_C0603_1uF; footprint Capacitor_SMD:C_0603_1608Metric -> 0WJQ:C_0603_WJQ; symbol 0WJQ:03.0011_C0603_1uF -> 0WJQ:03.4001_C0603_1uF; 编码 03.0011 -> 03.4001
- C33: value 03.0012_C0603_2.2uF -> 03.4002_C0603_2.2uF; footprint Capacitor_SMD:C_0603_1608Metric -> 0WJQ:C_0603_WJQ; symbol 0WJQ:03.0012_C0603_2.2uF -> 0WJQ:03.4002_C0603_2.2uF; 编码 03.0012 -> 03.4002
- C34, C36, C37: footprint Capacitor_SMD:C_0402_1005Metric -> 0WJQ:C_0402_WJQ
- R13, R14, R15, R16, R17, R18, R19, R20: footprint Resistor_SMD:R_0402_1005Metric -> 0WJQ:R_0402_WJQ
Connections:
- no-connect marks 19 -> 20
Changed lines of the file:
@@
 	1900 2550 1900 1050
 $Comp
-L 0WJQ:03.0011_C0603_1uF C31
+L 0WJQ:03.4001_C0603_1uF C31
 U 1 1 5E3BC13F
 P 1350 2650
+AR Path="/5E3BC13F" Ref="C31"  Part="1"
+AR Path="/5E3A651C/5E3BC13F" Ref="C31"  Part="1"
 F 0 "C31" H 1442 2696 50  0000 L CNN
-F 1 "03.0011_C0603_1uF" H 1360 2570 50  0001 L CNN
-F 2 "Capacitor_SMD:C_0603_1608Metric" H 750 2600 50  0001 C CNN
+F 1 "03.4001_C0603_1uF" H 1360 2570 50  0001 L CNN
+F 2 "0WJQ:C_0603_WJQ" H 750 2600 50  0001 C CNN
 F 3 "~" H 1350 2650 50  0001 C CNN
 F 4 "贴片瓷片电容" H 1350 2650 50  0001 C CNN "分类"
-F 5 "03.0011" H 1350 2650 50  0001 C CNN "编码"
+F 5 "03.4001" H 1350 2650 50  0001 C CNN "编码"
 F 6 "1uF,16V,K,0603,,X7R" H 1350 2650 50  0001 C CNN "规格"
 F 7 "1uF" H 1442 2605 50  0000 L CNN "参数"
@@
 F 0 "C34" H 2642 2046 50  0000 L CNN
 F 1 "03.0009_C0402_100nF" H 2560 1920 50  0001 L CNN
-F 2 "Capacitor_SMD:C_0402_1005Metric" H 1950 1950 50  0001 C CNN
+F 2 "0WJQ:C_0402_WJQ" H 1950 1950 50  0001 C CNN
 F 3 "~" H 2550 2000 50  0001 C CNN
 F 4 "贴片瓷片电容" H 2550 2000 50  0001 C CNN "分类"
@@
 $EndComp
 $Comp
-L 0WJQ:03.0012_C0603_2.2uF C33
+L 0WJQ:03.4002_C0603_2.2uF C33
 U 1 1 5E3BF31F
 P 2150 2000
+AR Path="/5E3BF31F" Ref="C33"  Part="1"
+AR Path="/5E3A651C/5E3BF31F" Ref="C33"  Part="1"
 F 0 "C33" H 2242 2046 50  0000 L CNN
-F 1 "03.0012_C0603_2.2uF" H 2160 1920 50  0001 L CNN
-F 2 "Capacitor_SMD:C_0603_1608Metric" H 1550 1950 50  0001 C CNN
+F 1 "03.4002_C0603_2.2uF" H 2160 1920 50  0001 L CNN
+F 2 "0WJQ:C_0603_WJQ" H 1550 1950 50  0001 C CNN
 F 3 "~" H 2150 2000 50  0001 C CNN
 F 4 "贴片瓷片电容" H 2150 2000 50  0001 C CNN "分类"
-F 5 "03.0012" H 2150 2000 50  0001 C CNN "编码"
+F 5 "03.4002" H 2150 2000 50  0001 C CNN "编码"
 F 6 "2.2uF,16V,K,X5R" H 2150 2000 50  0001 C CNN "规格"
 F 7 "2.2uF" H 2242 1955 50  0000 L CNN "参数"
@@
 F 0 "R18" H 3750 3857 50  0000 C CNN
 F 1 "02.0005_R0402_4K7_1%" H 3600 3840 50  0001 L BNN
-F 2 "Resistor_SMD:R_0402_1005Metric" H 3550 3410 50  0001 L BNN
+F 2 "0WJQ:R_0402_WJQ" H 3550 3410 50  0001 L BNN
 F 3 "" H 3550 3510 50  0001 L BNN
 F 4 "贴片电阻" H 3750 3650 50  0001 C CNN "分类"
@@
 F 0 "R17" V 3604 5570 50  0000 L CNN
 F 1 "02.0014_R0402_47K_1%" H 3500 5690 50  0001 L BNN
-F 2 "Resistor_SMD:R_0402_1005Metric" H 3450 5260 50  0001 L BNN
+F 2 "0WJQ:R_0402_WJQ" H 3450 5260 50  0001 L BNN
 F 3 "" H 3450 5360 50  0001 L BNN
 F 4 "贴片电阻" H 3650 5500 50  0001 C CNN "分类"
@@
 F 0 "R15" V 2804 5570 50  0000 L CNN
 F 1 "02.0014_R0402_47K_1%" H 2700 5690 50  0001 L BNN
-F 2 "Resistor_SMD:R_0402_1005Metric" H 2650 5260 50  0001 L BNN
+F 2 "0WJQ:R_0402_WJQ" H 2650 5260 50  0001 L BNN
 F 3 "" H 2650 5360 50  0001 L BNN
 F 4 "贴片电阻" H 2850 5500 50  0001 C CNN "分类"
@@
 F 0 "R14" V 2404 5570 50  0000 L CNN
 F 1 "02.0014_R0402_47K_1%" H 2300 5690 50  0001 L BNN
-F 2 "Resistor_SMD:R_0402_1005Metric" H 2250 5260 50  0001 L BNN
+F 2 "0WJQ:R_0402_WJQ" H 2250 5260 50  0001 L BNN
 F 3 "" H 2250 5360 50  0001 L BNN
 F 4 "贴片电阻" H 2450 5500 50  0001 C CNN "分类"
@@
 F 0 "R13" V 2004 5570 50  0000 L CNN
 F 1 "02.0014_R0402_47K_1%" H 1900 5690 50  0001 L BNN
-F 2 "Resistor_SMD:R_0402_1005Metric" H 1850 5260 50  0001 L BNN
+F 2 "0WJQ:R_0402_WJQ" H 1850 5260 50  0001 L BNN
 F 3 "" H 1850 5360 50  0001 L BNN
 F 4 "贴片电阻" H 2050 5500 50  0001 C CNN "分类"
@@
 F 0 "C36" H 3392 6946 50  0000 L CNN
 F 1 "03.0009_C0402_100nF" H 3310 6820 50  0001 L CNN
-F 2 "Capacitor_SMD:C_0402_1005Metric" H 2700 6850 50  0001 C CNN
+F 2 "0WJQ:C_0402_WJQ" H 2700 6850 50  0001 C CNN
 F 3 "~" H 3300 6900 50  0001 C CNN
 F 4 "贴片瓷片电容" H 3300 6900 50  0001 C CNN "分类"
@@
 F 0 "R20" V 8546 2530 50  0000 R CNN
 F 1 "02.0008_R0402_10K_1%" H 8350 2790 50  0001 L BNN
-F 2 "Resistor_SMD:R_0402_1005Metric" H 8300 2360 50  0001 L BNN
+F 2 "0WJQ:R_0402_WJQ" H 8300 2360 50  0001 L BNN
 F 3 "" H 8300 2460 50  0001 L BNN
 F 4 "贴片电阻" H 8500 2600 50  0001 C CNN "分类"
@@
 F 0 "R19" H 5550 1807 50  0000 C CNN
 F 1 "02.0008_R0402_10K_1%" H 5400 1790 50  0001 L BNN
-F 2 "Resistor_SMD:R_0402_1005Metric" H 5350 1360 50  0001 L BNN
+F 2 "0WJQ:R_0402_WJQ" H 5350 1360 50  0001 L BNN
 F 3 "" H 5350 1460 50  0001 L BNN
 F 4 "贴片电阻" H 5550 1600 50  0001 C CNN "分类"
@@
 F 0 "R16" V 3254 5570 50  0000 L CNN
 F 1 "02.0014_R0402_47K_1%" H 3150 5690 50  0001 L BNN
-F 2 "Resistor_SMD:R_0402_1005Metric" H 3100 5260 50  0001 L BNN
+F 2 "0WJQ:R_0402_WJQ" H 3100 5260 50  0001 L BNN
 F 3 "" H 3100 5360 50  0001 L BNN
 F 4 "贴片电阻" H 3300 5500 50  0001 C CNN "分类"
@@
 F 0 "C37" V 6121 1250 50  0000 C CNN
 F 1 "03.0009_C0402_100nF" H 6360 1070 50  0001 L CNN
-F 2 "Capacitor_SMD:C_0402_1005Metric" H 6400 1200 50  0001 C CNN
+F 2 "0WJQ:C_0402_WJQ" H 6400 1200 50  0001 C CNN
 F 3 "~" H 6350 1250 50  0001 C CNN
 F 4 "贴片瓷片电容" H 6350 1250 50  0001 C CNN "分类"
@@
 	8950 5250 9200 5250
 Wire Wire Line
-	8950 5350 9200 5350
-Wire Wire Line
 	8950 5450 9200 5450
 Wire Wire Line
@@
 Wire Wire Line
 	9700 5550 10000 5550
-Wire Wire Line
-	10000 5350 9700 5350
 $Comp
 L power:+3V3 #PWR067
@@
 	9700 4850 10000 4850
 Wire Wire Line
-	9700 5050 10000 5050
-Wire Wire Line
 	9700 5150 10000 5150
-Wire Wire Line
-	10000 4950 9700 4950
 $Comp
 L power:GND #PWR060
@@
 Text HLabel 10000 4250 2    50   Output ~ 0
 SPI0_CLK
-NoConn ~ 10000 4950
-NoConn ~ 10000 5050
 Wire Wire Line
 	8600 4450 9200 4450
@@
 Wire Wire Line
 	9700 4750 10100 4750
-NoConn ~ 10000 5350
-NoConn ~ 8950 5350
 Text Notes 10000 4050 0    79   ~ 16
 PCB edge
@@
 Wire Wire Line
 	8750 1900 10050 1900
+NoConn ~ 2050 3850
+NoConn ~ 9700 4950
+NoConn ~ 9700 5050
+NoConn ~ 9700 5350
+NoConn ~ 9200 5350
 $EndSCHEMATC
