File: Power.sch (KiCad schematic (older format))
At the start: 30 parts, among them U2 09.0103_XC6206, U3 09.0102_EA3036

Commit message: 修改XC6206信息，明确型号为3.0V输出
Parts:
- U2: symbol 0WJQ:09.0103_XC6206 -> 0WJQ:09.0103_XC6206P302MR; 参数 XC6206 -> XC6206P302MR; 规格 XC6206 -> XC6206P302MR, 3.0V，250mA，12VinMax
Changed lines of the file:
@@
 	8850 2650 8850 2500
 $Comp
-L 0WJQ:09.0103_XC6206 U2
+L 0WJQ:09.0103_XC6206P302MR U2
 U 1 1 5E4D75C1
 P 2400 4100
+AR Path="/5E4D75C1" Ref="U2"  Part="1"
+AR Path="/5E3A4AC6/5E4D75C1" Ref="U2"  Part="1"
 F 0 "U2" H 2400 4342 50  0000 C CNN
 F 1 "09.0103_XC6206" H 2400 4225 50  0001 L CNN
 F 2 "Package_TO_SOT_SMD:SOT-23" H 2400 4325 50  0001 C CIN
-F 3 "http://www.tme.eu/fr/Document/ced3461ed31ea70a3c416fb648e0cde7/APE8865-3.pdf" H 2400 4100 50  0001 C CNN
+F 3 "https://item.szlcsc.com/10507.html" H 2400 4100 50  0001 C CNN
 F 4 "LDO" H 2400 4100 50  0001 C CNN "分类"
 F 5 "09.0103" H 2400 4100 50  0001 C CNN "编码"
-F 6 "XC6206" H 2400 4100 50  0001 C CNN "规格"
-F 7 "XC6206" H 2400 4251 50  0000 C CNN "参数"
+F 6 "XC6206P302MR, 3.0V，250mA，12VinMax" H 2400 4100 50  0001 C CNN "规格"
+F 7 "XC6206P302MR" H 2050 3850 50  0000 C CNN "参数"
 	1    2400 4100
 	1    0    0    -1

Commit message: 优化封装外形丝印，PCB进行拼板处理
Parts:
- C19: value 03.0015_C0603_4.7uF -> 03.4004_C0603_10uF; footprint Capacitor_SMD:C_0603_1608Metric -> 0WJQ:C_0603_WJQ; symbol 0WJQ:03.0015_C0603_4.7uF -> 0WJQ:03.4004_C0603_10uF; 参数 4.7uF -> 10uF; 编码 03.0015 -> 03.4004; 规格 4.7uF,16V,K,0603,X5R -> 10uF,16V,K,0603,X5R
- C20, C24, C25, C26: footprint Capacitor_SMD:C_0402_1005Metric -> 0WJQ:C_0402_WJQ
- C21, C22, C23, C27, C28, C29: value 03.0016_C0603_10uF -> 03.4004_C0603_10uF; footprint Capacitor_SMD:C_0603_1608Metric -> 0WJQ:C_0603_WJQ; symbol 0WJQ:03.0016_C0603_10uF -> 0WJQ:03.4004_C0603_10uF; 编码 03.0016 -> 03.4004
- L1, L2, L3: footprint Inductor_SMD:L_1008_2520Metric -> 0WJQ:L_1008_2520_WJQ
- R10, R11, R4, R5, R6, R7, R8, R9: footprint Resistor_SMD:R_0402_1005Metric -> 0WJQ:R_0402_WJQ
Changed lines of the file:
@@
 F 0 "L1" H 5450 3090 50  0000 C CNN
 F 1 "06.0102_L2520_2.2uH" H 5450 2975 50  0001 C CNN
-F 2 "Inductor_SMD:L_1008_2520Metric" H 5350 2750 50  0001 C CNN
+F 2 "0WJQ:L_1008_2520_WJQ" H 5350 2750 50  0001 C CNN
 F 3 "~" V 5450 2900 50  0001 C CNN
 F 4 "贴片功率电感" H 5450 2850 50  0001 C CNN "分类"
@@
 F 0 "L2" H 5450 3590 50  0000 C CNN
 F 1 "06.0102_L2520_2.2uH" H 5450 3475 50  0001 C CNN
-F 2 "Inductor_SMD:L_1008_2520Metric" H 5350 3250 50  0001 C CNN
+F 2 "0WJQ:L_1008_2520_WJQ" H 5350 3250 50  0001 C CNN
 F 3 "~" V 5450 3400 50  0001 C CNN
 F 4 "贴片功率电感" H 5450 3350 50  0001 C CNN "分类"
@@
 F 0 "L3" H 5450 4090 50  0000 C CNN
 F 1 "06.0102_L2520_2.2uH" H 5450 3975 50  0001 C CNN
-F 2 "Inductor_SMD:L_1008_2520Metric" H 5350 3750 50  0001 C CNN
+F 2 "0WJQ:L_1008_2520_WJQ" H 5350 3750 50  0001 C CNN
 F 3 "~" V 5450 3900 50  0001 C CNN
 F 4 "贴片功率电感" H 5450 3850 50  0001 C CNN "分类"
@@
 $EndComp
 $Comp
-L 0WJQ:03.0016_C0603_10uF C21
+L 0WJQ:03.4004_C0603_10uF C21
 U 1 1 5E3DD939
 P 4100 3000
+AR Path="/5E3DD939" Ref="C21"  Part="1"
+AR Path="/5E3A4AC6/5E3DD939" Ref="C21"  Part="1"
 F 0 "C21" H 4192 3046 50  0000 L CNN
-F 1 "03.0016_C0603_10uF" H 4110 2920 50  0001 L CNN
-F 2 "Capacitor_SMD:C_0603_1608Metric" H 3500 2950 50  0001 C CNN
+F 1 "03.4004_C0603_10uF" H 4110 2920 50  0001 L CNN
+F 2 "0WJQ:C_0603_WJQ" H 3500 2950 50  0001 C CNN
 F 3 "~" H 4100 3000 50  0001 C CNN
 F 4 "贴片瓷片电容" H 4100 3000 50  0001 C CNN "分类"
-F 5 "03.0016" H 4100 3000 50  0001 C CNN "编码"
+F 5 "03.4004" H 4100 3000 50  0001 C CNN "编码"
 F 6 "10uF,16V,K,0603,X5R" H 4100 3000 50  0001 C CNN "规格"
 F 7 "10uF" H 4192 2955 50  0000 L CNN "参数"
@@
 $EndComp
 $Comp
-L 0WJQ:03.0016_C0603_10uF C22
+L 0WJQ:03.4004_C0603_10uF C22
 U 1 1 5E3DE492
 P 4100 3500
+AR Path="/5E3DE492" Ref="C22"  Part="1"
+AR Path="/5E3A4AC6/5E3DE492" Ref="C22"  Part="1"
 F 0 "C22" H 4192 3546 50  0000 L CNN
-F 1 "03.0016_C0603_10uF" H 4110 3420 50  0001 L CNN
-F 2 "Capacitor_SMD:C_0603_1608Metric" H 3500 3450 50  0001 C CNN
+F 1 "03.4004_C0603_10uF" H 4110 3420 50  0001 L CNN
+F 2 "0WJQ:C_0603_WJQ" H 3500 3450 50  0001 C CNN
 F 3 "~" H 4100 3500 50  0001 C CNN
 F 4 "贴片瓷片电容" H 4100 3500 50  0001 C CNN "分类"
-F 5 "03.0016" H 4100 3500 50  0001 C CNN "编码"
+F 5 "03.4004" H 4100 3500 50  0001 C CNN "编码"
 F 6 "10uF,16V,K,0603,X5R" H 4100 3500 50  0001 C CNN "规格"
 F 7 "10uF" H 4192 3455 50  0000 L CNN "参数"
@@
 $EndComp
 $Comp
-L 0WJQ:03.0016_C0603_10uF C23
+L 0WJQ:03.4004_C0603_10uF C23
 U 1 1 5E3DEC88
 P 4100 4000
+AR Path="/5E3DEC88" Ref="C23"  Part="1"
+AR Path="/5E3A4AC6/5E3DEC88" Ref="C23"  Part="1"
 F 0 "C23" H 4192 4046 50  0000 L CNN
-F 1 "03.0016_C0603_10uF" H 4110 3920 50  0001 L CNN
-F 2 "Capacitor_SMD:C_0603_1608Metric" H 3500 3950 50  0001 C CNN
+F 1 "03.4004_C0603_10uF" H 4110 3920 50  0001 L CNN
+F 2 "0WJQ:C_0603_WJQ" H 3500 3950 50  0001 C CNN
 F 3 "~" H 4100 4000 50  0001 C CNN
 F 4 "贴片瓷片电容" H 4100 4000 50  0001 C CNN "分类"
-F 5 "03.0016" H 4100 4000 50  0001 C CNN "编码"
+F 5 "03.4004" H 4100 4000 50  0001 C CNN "编码"
 F 6 "10uF,16V,K,0603,X5R" H 4100 4000 50  0001 C CNN "规格"
 F 7 "10uF" H 4192 3955 50  0000 L CNN "参数"
@@
 F 0 "C24" H 4542 3046 50  0000 L CNN
 F 1 "03.0009_C0402_100nF" H 4460 2820 50  0001 L CNN
-F 2 "Capacitor_SMD:C_0402_1005Metric" H 4500 2950 50  0001 C CNN
+F 2 "0WJQ:C_0402_WJQ" H 4500 2950 50  0001 C CNN
 F 3 "~" H 4450 3000 50  0001 C CNN
 F 4 "贴片瓷片电容" H 4450 3000 50  0001 C CNN "分类"
@@
 F 0 "C25" H 4542 3546 50  0000 L CNN
 F 1 "03.0009_C0402_100nF" H 4460 3320 50  0001 L CNN
-F 2 "Capacitor_SMD:C_0402_1005Metric" H 4500 3450 50  0001 C CNN
+F 2 "0WJQ:C_0402_WJQ" H 4500 3450 50  0001 C CNN
 F 3 "~" H 4450 3500 50  0001 C CNN
 F 4 "贴片瓷片电容" H 4450 3500 50  0001 C CNN "分类"
@@
 F 0 "C26" H 4542 4046 50  0000 L CNN
 F 1 "03.0009_C0402_100nF" H 4460 3820 50  0001 L CNN
-F 2 "Capacitor_SMD:C_0402_1005Metric" H 4500 3950 50  0001 C CNN
+F 2 "0WJQ:C_0402_WJQ" H 4500 3950 50  0001 C CNN
 F 3 "~" H 4450 4000 50  0001 C CNN
 F 4 "贴片瓷片电容" H 4450 4000 50  0001 C CNN "分类"
@@
 F 0 "R8" H 4800 4607 50  0000 C CNN
 F 1 "02.0023_R0402_150K_1%" H 4650 4590 50  0001 L BNN
-F 2 "Resistor_SMD:R_0402_1005Metric" H 4600 4160 50  0001 L BNN
+F 2 "0WJQ:R_0402_WJQ" H 4600 4160 50  0001 L BNN
 F 3 "" H 4600 4260 50  0001 L BNN
 F 4 "贴片电阻" H 4800 4400 50  0001 C CNN "分类"
@@
 F 0 "R10" H 5150 3807 50  0000 C CNN
 F 1 "02.0024_R0402_470K_1%" H 5000 3790 50  0001 L BNN
-F 2 "Resistor_SMD:R_0402_1005Metric" H 4950 3360 50  0001 L BNN
+F 2 "0WJQ:R_0402_WJQ" H 4950 3360 50  0001 L BNN
 F 3 "" H 4950 3460 50  0001 L BNN
 F 4 "贴片电阻" H 5150 3600 50  0001 C CNN "分类"
@@
 F 0 "R9" H 5150 3307 50  0000 C CNN
 F 1 "02.0025_R0402_680K_1%" H 5000 3290 50  0001 L BNN
-F 2 "Resistor_SMD:R_0402_1005Metric" H 4950 2860 50  0001 L BNN
+F 2 "0WJQ:R_0402_WJQ" H 4950 2860 50  0001 L BNN
 F 3 "" H 4950 2960 50  0001 L BNN
 F 4 "贴片电阻" H 5150 3100 50  0001 C CNN "分类"
@@
 F 0 "R6" H 4800 3507 50  0000 C CNN
 F 1 "02.0023_R0402_150K_1%" H 4650 3490 50  0001 L BNN
-F 2 "Resistor_SMD:R_0402_1005Metric" H 4600 3060 50  0001 L BNN
+F 2 "0WJQ:R_0402_WJQ" H 4600 3060 50  0001 L BNN
 F 3 "" H 4600 3160 50  0001 L BNN
 F 4 "贴片电阻" H 4800 3300 50  0001 C CNN "分类"
@@
 F 0 "R11" H 5150 4307 50  0000 C CNN
 F 1 "02.0023_R0402_150K_1%" H 5000 4290 50  0001 L BNN
-F 2 "Resistor_SMD:R_0402_1005Metric" H 4950 3860 50  0001 L BNN
+F 2 "0WJQ:R_0402_WJQ" H 4950 3860 50  0001 L BNN
 F 3 "" H 4950 3960 50  0001 L BNN
 F 4 "贴片电阻" H 5150 4100 50  0001 C CNN "分类"
@@
 F 0 "R7" H 4800 4007 50  0000 C CNN
 F 1 "02.0023_R0402_150K_1%" H 4650 3990 50  0001 L BNN
-F 2 "Resistor_SMD:R_0402_1005Metric" H 4600 3560 50  0001 L BNN
+F 2 "0WJQ:R_0402_WJQ" H 4600 3560 50  0001 L BNN
 F 3 "" H 4600 3660 50  0001 L BNN
 F 4 "贴片电阻" H 4800 3800 50  0001 C CNN "分类"
@@
 $EndComp
 $Comp
-L 0WJQ:03.0015_C0603_4.7uF C19
+L 0WJQ:03.4004_C0603_10uF C19
 U 1 1 5E4DB6A2
 P 2850 4200
+AR Path="/5E4DB6A2" Ref="C19"  Part="1"
+AR Path="/5E3A4AC6/5E4DB6A2" Ref="C19"  Part="1"
 F 0 "C19" H 2942 4246 50  0000 L CNN
-F 1 "03.0015_C0603_4.7uF" H 2860 4020 50  0001 L CNN
-F 2 "Capacitor_SMD:C_0603_1608Metric" H 2250 4150 50  0001 C CNN
+F 1 "03.4004_C0603_10uF" H 2860 4020 50  0001 L CNN
+F 2 "0WJQ:C_0603_WJQ" H 2250 4150 50  0001 C CNN
 F 3 "~" H 2850 4200 50  0001 C CNN
 F 4 "贴片瓷片电容" H 2850 4100 50  0001 C CNN "分类"
-F 5 "03.0015" H 2850 4100 50  0001 C CNN "编码"
-F 6 "4.7uF,16V,K,0603,X5R" H 2850 4100 50  0001 C CNN "规格"
-F 7 "4.7uF" H 2942 4155 50  0000 L CNN "参数"
+F 5 "03.4004" H 2850 4100 50  0001 C CNN "编码"
+F 6 "10uF,16V,K,0603,X5R" H 2850 4100 50  0001 C CNN "规格"
+F 7 "10uF" H 2942 4155 50  0000 L CNN "参数"
 	1    2850 4200
 	1    0    0    -1
@@
 F 0 "C20" H 3342 4246 50  0000 L CNN
 F 1 "03.0009_C0402_100nF" H 3260 4020 50  0001 L CNN
-F 2 "Capacitor_SMD:C_0402_1005Metric" H 3300 4150 50  0001 C CNN
+F 2 "0WJQ:C_0402_WJQ" H 3300 4150 50  0001 C CNN
 F 3 "~" H 3250 4200 50  0001 C CNN
 F 4 "贴片瓷片电容" H 3250 4200 50  0001 C CNN "分类"
@@
 Connection ~ 3250 4100
 $Comp
-L 0WJQ:03.0016_C0603_10uF C27
+L 0WJQ:03.4004_C0603_10uF C27
 U 1 1 5E837CF1
 P 7150 3000
+AR Path="/5E837CF1" Ref="C27"  Part="1"
+AR Path="/5E3A4AC6/5E837CF1" Ref="C27"  Part="1"
 F 0 "C27" H 7242 3046 50  0000 L CNN
-F 1 "03.0016_C0603_10uF" H 7160 2920 50  0001 L CNN
-F 2 "Capacitor_SMD:C_0603_1608Metric" H 6550 2950 50  0001 C CNN
+F 1 "03.4004_C0603_10uF" H 7160 2920 50  0001 L CNN
+F 2 "0WJQ:C_0603_WJQ" H 6550 2950 50  0001 C CNN
 F 3 "~" H 7150 3000 50  0001 C CNN
 F 4 "贴片瓷片电容" H 7150 3000 50  0001 C CNN "分类"
-F 5 "03.0016" H 7150 3000 50  0001 C CNN "编码"
+F 5 "03.4004" H 7150 3000 50  0001 C CNN "编码"
 F 6 "10uF,16V,K,0603,X5R" H 7150 3000 50  0001 C CNN "规格"
 F 7 "10uF" H 7242 2955 50  0000 L CNN "参数"
@@
 $EndComp
 $Comp
-L 0WJQ:03.0016_C0603_10uF C28
+L 0WJQ:03.4004_C0603_10uF C28
 U 1 1 5E83CA71
 P 7550 3000
+AR Path="/5E83CA71" Ref="C28"  Part="1"
+AR Path="/5E3A4AC6/5E83CA71" Ref="C28"  Part="1"
 F 0 "C28" H 7642 3046 50  0000 L CNN
-F 1 "03.0016_C0603_10uF" H 7560 2920 50  0001 L CNN
-F 2 "Capacitor_SMD:C_0603_1608Metric" H 6950 2950 50  0001 C CNN
+F 1 "03.4004_C0603_10uF" H 7560 2920 50  0001 L CNN
+F 2 "0WJQ:C_0603_WJQ" H 6950 2950 50  0001 C CNN
 F 3 "~" H 7550 3000 50  0001 C CNN
 F 4 "贴片瓷片电容" H 7550 3000 50  0001 C CNN "分类"
-F 5 "03.0016" H 7550 3000 50  0001 C CNN "编码"
+F 5 "03.4004" H 7550 3000 50  0001 C CNN "编码"
 F 6 "10uF,16V,K,0603,X5R" H 7550 3000 50  0001 C CNN "规格"
 F 7 "10uF" H 7642 2955 50  0000 L CNN "参数"
@@
 $EndComp
 $Comp
-L 0WJQ:03.0016_C0603_10uF C29
+L 0WJQ:03.4004_C0603_10uF C29
 U 1 1 5E83D2F8
 P 7900 3000
+AR Path="/5E83D2F8" Ref="C29"  Part="1"
+AR Path="/5E3A4AC6/5E83D2F8" Ref="C29"  Part="1"
 F 0 "C29" H 7992 3046 50  0000 L CNN
-F 1 "03.0016_C0603_10uF" H 7910 2920 50  0001 L CNN
-F 2 "Capacitor_SMD:C_0603_1608Metric" H 7300 2950 50  0001 C CNN
+F 1 "03.4004_C0603_10uF" H 7910 2920 50  0001 L CNN
+F 2 "0WJQ:C_0603_WJQ" H 7300 2950 50  0001 C CNN
 F 3 "~" H 7900 3000 50  0001 C CNN
 F 4 "贴片瓷片电容" H 7900 3000 50  0001 C CNN "分类"
-F 5 "03.0016" H 7900 3000 50  0001 C CNN "编码"
+F 5 "03.4004" H 7900 3000 50  0001 C CNN "编码"
 F 6 "10uF,16V,K,0603,X5R" H 7900 3000 50  0001 C CNN "规格"
 F 7 "10uF" H 7992 2955 50  0000 L CNN "参数"
@@
 F 0 "R5" H 3700 4193 50  0000 C CNN
 F 1 "02.0001_R0402_0R_1%" H 3550 4640 50  0001 L BNN
-F 2 "Resistor_SMD:R_0402_1005Metric" H 3500 4160 50  0001 L BNN
+F 2 "0WJQ:R_0402_WJQ" H 3500 4160 50  0001 L BNN
 F 3 "" H 3500 4260 50  0001 L BNN
 F 4 "贴片电阻" H 3700 4400 50  0001 C CNN "分类"
@@
 F 0 "R4" V 2704 3220 50  0000 L CNN
 F 1 "02.0003_R0402_1K_1%" H 2600 3340 50  0001 L BNN
-F 2 "Resistor_SMD:R_0402_1005Metric" H 2550 2910 50  0001 L BNN
+F 2 "0WJQ:R_0402_WJQ" H 2550 2910 50  0001 L BNN
 F 3 "" H 2550 3010 50  0001 L BNN
 F 4 "贴片电阻" H 2750 3150 50  0001 C CNN "分类"
