File: TV.sch (KiCad schematic (older format))
At the start: 11 parts, among them J6 10.0202_PH2X9_2D54_V

Commit message: 优化封装外形丝印，PCB进行拼板处理
Parts:
- C38, C40, C42: footprint Capacitor_SMD:C_0402_1005Metric -> 0WJQ:C_0402_WJQ
- C39, C43, C45: value 03.0015_C0603_4.7uF -> 03.4003_C0603_4.7uF; footprint Capacitor_SMD:C_0603_1608Metric -> 0WJQ:C_0603_WJQ; symbol 0WJQ:03.0015_C0603_4.7uF -> 0WJQ:03.4003_C0603_4.7uF; 编码 03.0015 -> 03.4003
- C41: value 03.0016_C0603_10uF -> 03.4004_C0603_10uF; footprint Capacitor_SMD:C_0603_1608Metric -> 0WJQ:C_0603_WJQ; symbol 0WJQ:03.0016_C0603_10uF -> 0WJQ:03.4004_C0603_10uF; 编码 03.0016 -> 03.4004
- C44: symbol 0WJQ:03.0016_C0603_10uF -> F1C200S_KIT-rescue:03.0016_C0603_10uF-0WJQ
- R21, R22: footprint Resistor_SMD:R_0402_1005Metric -> 0WJQ:R_0402_WJQ
Changed lines of the file:
@@
 $EndDescr
 $Comp
-L 0WJQ:03.0015_C0603_4.7uF C?
+L 0WJQ:03.4003_C0603_4.7uF C?
 U 1 1 5E6BBBD7
 P 8400 2700
 AR Path="/5E3A4A8E/5E6BBBD7" Ref="C?"  Part="1"
 AR Path="/5E5BEA7B/5E6BBBD7" Ref="C43"  Part="1"
+AR Path="/5E6BBBD7" Ref="C43"  Part="1"
 F 0 "C43" H 8492 2746 50  0000 L CNN
-F 1 "03.0015_C0603_4.7uF" H 8410 2520 50  0001 L CNN
-F 2 "Capacitor_SMD:C_0603_1608Metric" H 7800 2650 50  0001 C CNN
+F 1 "03.4003_C0603_4.7uF" H 8410 2520 50  0001 L CNN
+F 2 "0WJQ:C_0603_WJQ" H 7800 2650 50  0001 C CNN
 F 3 "~" H 8400 2700 50  0001 C CNN
 F 4 "贴片瓷片电容" H 8400 2600 50  0001 C CNN "分类"
-F 5 "03.0015" H 8400 2600 50  0001 C CNN "编码"
+F 5 "03.4003" H 8400 2600 50  0001 C CNN "编码"
 F 6 "4.7uF,16V,K,0603,X5R" H 8400 2600 50  0001 C CNN "规格"
 F 7 "4.7uF" H 8492 2655 50  0000 L CNN "参数"
@@
 	8400 2900 8400 2800
 $Comp
-L 0WJQ:03.0016_C0603_10uF C?
+L 0WJQ:03.4004_C0603_10uF C?
 U 1 1 5E6BBBF2
 P 7400 2600
@@
 AR Path="/5E3A4A8E/5E6BBBF2" Ref="C?"  Part="1"
 AR Path="/5E5BEA7B/5E6BBBF2" Ref="C41"  Part="1"
+AR Path="/5E6BBBF2" Ref="C41"  Part="1"
 F 0 "C41" H 7492 2646 50  0000 L CNN
-F 1 "03.0016_C0603_10uF" H 7410 2520 50  0001 L CNN
-F 2 "Capacitor_SMD:C_0603_1608Metric" H 6800 2550 50  0001 C CNN
+F 1 "03.4004_C0603_10uF" H 7410 2520 50  0001 L CNN
+F 2 "0WJQ:C_0603_WJQ" H 6800 2550 50  0001 C CNN
 F 3 "~" H 7400 2600 50  0001 C CNN
 F 4 "贴片瓷片电容" H 7400 2600 50  0001 C CNN "分类"
-F 5 "03.0016" H 7400 2600 50  0001 C CNN "编码"
+F 5 "03.4004" H 7400 2600 50  0001 C CNN "编码"
 F 6 "10uF,16V,K,0603,X5R" H 7400 2600 50  0001 C CNN "规格"
 F 7 "10uF" H 7492 2555 50  0000 L CNN "参数"
@@
 F 0 "C42" H 7842 2646 50  0000 L CNN
 F 1 "03.0009_C0402_100nF" H 7760 2420 50  0001 L CNN
-F 2 "Capacitor_SMD:C_0402_1005Metric" H 7800 2550 50  0001 C CNN
+F 2 "0WJQ:C_0402_WJQ" H 7800 2550 50  0001 C CNN
 F 3 "~" H 7750 2600 50  0001 C CNN
 F 4 "贴片瓷片电容" H 7750 2600 50  0001 C CNN "分类"
@@
 F 0 "R22" H 7050 2607 50  0000 C CNN
 F 1 "02.0001_R0402_0R_1%" H 6900 2640 50  0001 L BNN
-F 2 "Resistor_SMD:R_0402_1005Metric" H 6850 2160 50  0001 L BNN
+F 2 "0WJQ:R_0402_WJQ" H 6850 2160 50  0001 L BNN
 F 3 "" H 6850 2260 50  0001 L BNN
 F 4 "贴片电阻" H 7050 2400 50  0001 C CNN "分类"
@@
 F 0 "C38" H 3692 2646 50  0000 L CNN
 F 1 "03.0001_C0402_1uF" H 3660 2270 50  0001 L CNN
-F 2 "Capacitor_SMD:C_0402_1005Metric" H 3600 2200 50  0001 C CNN
+F 2 "0WJQ:C_0402_WJQ" H 3600 2200 50  0001 C CNN
 F 3 "~" H 3600 2600 50  0001 C CNN
 F 4 "贴片瓷片电容" H 3700 2100 50  0001 C CNN "分类"
@@
 $EndComp
 $Comp
-L 0WJQ:03.0015_C0603_4.7uF C39
+L 0WJQ:03.4003_C0603_4.7uF C39
 U 1 1 5EC51247
 P 4050 2600
+AR Path="/5EC51247" Ref="C39"  Part="1"
+AR Path="/5E5BEA7B/5EC51247" Ref="C39"  Part="1"
 F 0 "C39" H 4142 2646 50  0000 L CNN
-F 1 "03.0015_C0603_4.7uF" H 4060 2420 50  0001 L CNN
-F 2 "Capacitor_SMD:C_0603_1608Metric" H 3450 2550 50  0001 C CNN
+F 1 "03.4003_C0603_4.7uF" H 4060 2420 50  0001 L CNN
+F 2 "0WJQ:C_0603_WJQ" H 3450 2550 50  0001 C CNN
 F 3 "~" H 4050 2600 50  0001 C CNN
 F 4 "贴片瓷片电容" H 4050 2500 50  0001 C CNN "分类"
-F 5 "03.0015" H 4050 2500 50  0001 C CNN "编码"
+F 5 "03.4003" H 4050 2500 50  0001 C CNN "编码"
 F 6 "4.7uF,16V,K,0603,X5R" H 4050 2500 50  0001 C CNN "规格"
 F 7 "4.7uF" H 4142 2555 50  0000 L CNN "参数"
@@
 F 0 "C40" H 4542 2646 50  0000 L CNN
 F 1 "03.0009_C0402_100nF" H 4460 2420 50  0001 L CNN
-F 2 "Capacitor_SMD:C_0402_1005Metric" H 4500 2550 50  0001 C CNN
+F 2 "0WJQ:C_0402_WJQ" H 4500 2550 50  0001 C CNN
 F 3 "~" H 4450 2600 50  0001 C CNN
 F 4 "贴片瓷片电容" H 4450 2600 50  0001 C CNN "分类"
@@
 F 0 "R21" V 4804 2720 50  0000 L CNN
 F 1 "02.0027_R0402_200K_1%" H 4700 2840 50  0001 L BNN
-F 2 "Resistor_SMD:R_0402_1005Metric" H 4650 2410 50  0001 L BNN
+F 2 "0WJQ:R_0402_WJQ" H 4650 2410 50  0001 L BNN
 F 3 "" H 4650 2510 50  0001 L BNN
 F 4 "贴片电阻" H 4850 2650 50  0001 C CNN "分类"
@@
 	5950 4800 6300 4800
 $Comp
-L 0WJQ:03.0015_C0603_4.7uF C?
+L 0WJQ:03.4003_C0603_4.7uF C?
 U 1 1 5E6BBBCD
 P 8950 2700
 AR Path="/5E3A4A8E/5E6BBBCD" Ref="C?"  Part="1"
 AR Path="/5E5BEA7B/5E6BBBCD" Ref="C45"  Part="1"
+AR Path="/5E6BBBCD" Ref="C45"  Part="1"
 F 0 "C45" H 9042 2746 50  0000 L CNN
-F 1 "03.0015_C0603_4.7uF" H 8960 2520 50  0001 L CNN
-F 2 "Capacitor_SMD:C_0603_1608Metric" H 8350 2650 50  0001 C CNN
+F 1 "03.4003_C0603_4.7uF" H 8960 2520 50  0001 L CNN
+F 2 "0WJQ:C_0603_WJQ" H 8350 2650 50  0001 C CNN
 F 3 "~" H 8950 2700 50  0001 C CNN
 F 4 "贴片瓷片电容" H 8950 2600 50  0001 C CNN "分类"
-F 5 "03.0015" H 8950 2600 50  0001 C CNN "编码"
+F 5 "03.4003" H 8950 2600 50  0001 C CNN "编码"
 F 6 "4.7uF,16V,K,0603,X5R" H 8950 2600 50  0001 C CNN "规格"
 F 7 "4.7uF" H 9042 2655 50  0000 L CNN "参数"
@@
 $EndComp
 $Comp
-L 0WJQ:03.0016_C0603_10uF C?
+L F1C200S_KIT-rescue:03.0016_C0603_10uF-0WJQ C?
 U 1 1 5E6BBBE1
 P 8700 2500
@@
 AR Path="/5E3A4A8E/5E6BBBE1" Ref="C?"  Part="1"
 AR Path="/5E5BEA7B/5E6BBBE1" Ref="C44"  Part="1"
+AR Path="/5E6BBBE1" Ref="C44"  Part="1"
 F 0 "C44" H 8792 2546 50  0000 L CNN
 F 1 "03.0016_C0603_10uF" H 8710 2420 50  0001 L CNN
